Commit message: Simplified the world

File: src/my_robot/urdf/my_robot.xacro (robot description, xacro)
@@ -62,6 +62,6 @@
       <origin xyz="${x_reflect*wheel_xoff} ${y_reflect*(chassis_width/2+wheel_ygap)} ${-wheel_zoff}" rpy="0 0 0"/>
       <axis xyz="0 1 0"/>
-      <limit effort="10000" velocity="1000"/>
-      <dynamics damping="1.0" friction="1.0"/>
+      <limit effort="100" velocity="100"/>
+      <dynamics damping="0.1" friction="0.1"/>
     </joint>
   </xacro:macro>
@@ -90,6 +90,6 @@
     <origin xyz="0.0 0.0 ${-(wheel_radius+wheel_zoff)}" rpy="0 0 0"/>
   </joint>
-  <xacro:wheel prefix="drivewhl_l" x_reflect="-1" y_reflect="1" />
-  <xacro:wheel prefix="drivewhl_r" x_reflect="-1" y_reflect="-1" />
+  <xacro:wheel prefix="left" x_reflect="-1" y_reflect="1" />
+  <xacro:wheel prefix="right" x_reflect="-1" y_reflect="-1" />
   <!-- Caster Wheel -->
   <link name="front_caster">

Commit message: Troubleshooting

File: src/my_robot/urdf/my_robot.xacro (robot description, xacro)
@@ -81,5 +81,4 @@
       </geometry>
     </collision>
-    <xacro:box_inertia m="5" w="${chassis_width}" d="${chassis_length}" h="${chassis_height}"/>
   </link>
   <!-- Robot Footprint -->
@@ -116,5 +115,5 @@
   </joint>
   <!-- camera -->
-  <link name="camera1">
+  <link name="camera">
     <inertial>
       <mass value="${camera_mass}"/>
@@ -136,6 +135,6 @@
   </link>
   <joint type="fixed" name="camera_joint">
-    <origin xyz="${chassis_length/2 - camera_length} 0 ${chassis_height/2 + camera_height/2}" rpy="0 0 0"/>
-    <child link="camera1"/>
+    <origin xyz="${chassis_length/2} 0 ${-chassis_height/2 + camera_height}" rpy="0 0 0"/>
+    <child link="camera"/>
     <parent link="chassis"/>
     <axis xyz="0 1 0" rpy="0 0 0"/>
@@ -167,3 +166,16 @@
     <axis xyz="0 1 0" rpy="0 0 0"/>
   </joint>
+  <!-- Robot material/colour -->
+  <gazebo reference="camera">
+    <material>Gazebo/Red</material>
+  </gazebo>
+  <gazebo reference="chassis">
+    <material>Gazebo/Blue</material>
+  </gazebo>
+  <gazebo reference="left_wheel">
+    <material>Gazebo/Black</material>
+  </gazebo>
+  <gazebo reference="right_wheel">
+    <material>Gazebo/Black</material>
+  </gazebo>
 </robot>
